File: ESP_boards/ESP32/esp32s3_mini_pcb/esp32s3_mini_pcb.kicad_pcb (KiCad board)
At the start: 2 copper layers, 16 x 40.5 mm, 17 parts, among them J1 USB_B_Micro, U1 ESP32-S3-MINI-1, U2 D3V3XA4B10LP, U3 TLV75801PDRV

Commit message: Working on PCB
Parts:
- J1: footprint Connector_USB:USB_Micro-B_Amphenol_10103594-0001LF_Horizontal -> Connector_USB:USB_Micro-B_GCT_USB3076-30-A
- moved C5 46.4 mm to (96.0, 75.8), turned to 90 degrees
- moved C6 42.7 mm to (91.4, 75.8), turned to 90 degrees
- moved R1 39.9 mm to (48.5, 84.4)
- moved BOOT1 38.8 mm to (105.2, 83.5)
- moved U1 29.3 mm to (98.7, 62.6)
- moved U2 27.6 mm to (99.1, 85.1)
- moved J1 27.2 mm to (98.7, 89.1)
- moved R4 25.5 mm to (108.9, 77.2)
- moved C1 21.2 mm to (44.5, 81.9)
- moved D1 20.1 mm to (104.4, 75.7)
- moved C2 19.0 mm to (44.5, 84.4)
- moved U3 17.1 mm to (93.7, 77.2)
- moved C3 16.8 mm to (44.5, 86.9)
- moved RESET1 16.5 mm to (92.1, 83.5), turned to -90 degrees
- moved R3 14.9 mm to (95.3, 79.5)
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Routing:
- net /USB_P: track 0.00 -> 16.0 mm
- net /USB_N: track 0.00 -> 16.0 mm
- net Net-(U3-FB): track 0.00 -> 4.63 mm
- net /3V3: track 0.00 -> 4.32 mm
- net /5VUSB: track 0.00 -> 3.60 mm
Other:
- board outline removed

Commit message: Finished the board
Parts:
- moved C4 60.3 mm to (104.8, 88.4), turned to -90 degrees
- moved C2 59.5 mm to (103.8, 79.4)
- moved C1 59.4 mm to (103.8, 77.9)
- moved C3 48.0 mm to (92.5, 90.2), turned to 180 degrees
- moved R1 44.1 mm to (92.5, 88.5)
- moved R4 4.88 mm to (104.6, 75.0), turned to -90 degrees
- moved D1 1.68 mm to (102.9, 74.9), turned to 90 degrees
- moved RESET1 0.85 mm to (92.9, 83.5), turned to 90 degrees
- moved BOOT1 0.83 mm to (104.4, 83.5)
Connections:
- C3 pad 1: /EN -> /ESP_32EN
- R1 pad 2: /EN -> /ESP_32EN
- U1 pad 45: /EN -> /ESP_32EN
Routing:
- net /ESP_32EN: track 0.00 -> 38.1 mm, vias 0 -> 2
- net /3V3: track 4.32 -> 39.7 mm, vias 0 -> 2
- net /BOOT: track 0.00 -> 33.0 mm, vias 0 -> 2
- net Net-(D1-A): track 0.00 -> 1.68 mm
- added copper zone on B.Cu, net GND
- added copper zone on F.Cu, net GND
- added copper zone on In1.Cu, net GND
- added copper zone on In2.Cu, net GND
Other:
- board outline added: 17.7 x 34.4 mm
- copper layers 2 -> 4
