File: ESP_boards/ESP32/esp32s3_mini_pcb/esp32s3_mini_pcb.kicad_sch (KiCad schematic)
At the start: 0 parts

Commit message: ESP :: Work on the schematic
Parts:
- added BOOT1, RESET1: SW_MEC_5E, symbol Switch:SW_MEC_5E
- added C1, C3, C4: 0.1uF, symbol Device:C
- added C2: 10uF, symbol Device:C
- added J1: USB_B_Micro, symbol Connector:USB_B_Micro
- added R1: 10k, symbol Device:R
- added U1: ESP32-S3-MINI-1, RF_Module:ESP32-S2-MINI-1, symbol RF_Module:ESP32-S3-MINI-1
- added U2: D3V3XA4B10LP, Package_DFN_QFN:Diodes_UDFN-10_1.0x2.5mm_P0.5mm, symbol Power_Protection:D3V3XA4B10LP
- added U3: TLV75801PDRV, Package_SON:WSON-6-1EP_2x2mm_P0.65mm_EP1x1.6mm, symbol Regulator_Linear:TLV75801PDRV
Connections:
- new net: U3.3 (GND), U3.7 (GND)
- new net: U2.3 (VSS), U2.8 (VSS)
- new net 3V3: C1.1, C2.1, R1.1, U1.3 (3V3)
- new net BOOT: BOOT1.3 (K), BOOT1.4 (A), C4.1, U1.4 (IO0)
- new net EN: C3.1, R1.2, RESET1.3 (K), RESET1.4 (A), U1.45 (EN)
- new net GND: BOOT1.1, BOOT1.2, C1.2, C2.2, C3.2, C4.2, RESET1.1, RESET1.2, U1.1 (GND), U1.2 (GND), U1.42 (GND), U1.43 (GND), U1.46 (GND), U1.47 (GND), U1.48 (GND), U1.49 (GND), U1.50 (GND), U1.51 (GND), U1.52 (GND), U1.53 (GND), U1.54 (GND), U1.55 (GND), U1.56 (GND), U1.57 (GND), U1.58 (GND), U1.59 (GND), U1.60 (GND), U1.61 (GND), U1.62 (GND), U1.63 (GND), U1.64 (GND), U1.65 (GND)
- new net USB_N: U1.23 (USB_D-)
- new net USB_P: U1.24 (USB_D+)

Commit message: ESP :: Finished Schematic
Parts:
- added C5, C6: 10uF, symbol Device:C
- added D1: LED, symbol Device:LED
- added R2: 1M, symbol Device:R
- added R3: 200k, symbol Device:R
- added R4: 5.1k, symbol Device:R
Connections:
- net 3V3: now also U3.1 (OUT), C6.1, R2.1, R4.2
- net GND: now also J1.5 (GND), J1.6 (Shield), U2.3 (VSS), U2.8 (VSS), U3.3 (GND), U3.7 (GND), C5.2, C6.2, D1.1 (K), R3.2
- net USB_N: now also J1.2 (D-), U2.1, U2.10 (NC)
- net USB_P: now also J1.3 (D+), U2.2, U2.9 (NC)
- net at U3.2 (FB): now also R2.2, R3.1
- net 5VUSB: now reaches U3.4 (EN)
- net 5VUSB: now also J1.1 (VBUS), U2.4, U2.7 (NC), U3.6 (IN), C5.1
- new net: D1.2 (A), R4.1
- no-connect marks 0 -> 4

Commit message: ESP :: Laptop can't keep up, we will try at home
Parts:
- BOOT1, RESET1: footprint (none) -> Button_Switch_SMD:SW_SPST_PTS810
- C1, C2, C3, C4, C5, C6: footprint (none) -> Capacitor_SMD:C_0603_1608Metric
- D1: footprint (none) -> LED_SMD:LED_0603_1608Metric
- J1: footprint (none) -> Connector_USB:USB_Micro-B_Amphenol_10103594-0001LF_Horizontal
- R1, R2, R3, R4: footprint (none) -> Resistor_SMD:R_0603_1608Metric
Changed lines of the file:
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@@
 			)
 		)
-		(property "Footprint" ""
+		(property "Footprint" "Capacitor_SMD:C_0603_1608Metric"
 			(at 122.8852 118.11 0)
 			(effects
@@
 			)
 		)
-		(property "Footprint" ""
+		(property "Footprint" "Capacitor_SMD:C_0603_1608Metric"
 			(at 254.9652 55.88 0)
 			(effects
@@
 			)
 		)
-		(property "Footprint" ""
+		(property "Footprint" "Resistor_SMD:R_0603_1608Metric"
 			(at 155.702 127 90)
 			(effects
@@
 			)
 		)
-		(property "Footprint" ""
+		(property "Footprint" "Connector_USB:USB_Micro-B_Amphenol_10103594-0001LF_Horizontal"
 			(at 72.39 48.26 0)
 			(effects
@@
 			)
 		)
-		(property "Footprint" ""
+		(property "Footprint" "Capacitor_SMD:C_0603_1608Metric"
 			(at 167.3352 123.19 0)
 			(effects
@@
 			)
 		)
-		(property "Footprint" ""
+		(property "Footprint" "Button_Switch_SMD:SW_SPST_PTS810"
 			(at 137.16 33.02 0)
 			(effects
@@
 			)
 		)
-		(property "Footprint" ""
+		(property "Footprint" "Capacitor_SMD:C_0603_1608Metric"
 			(at 153.3652 73.66 0)
 			(effects
@@
 			)
 		)
-		(property "Footprint" ""
+		(property "Footprint" "Resistor_SMD:R_0603_1608Metric"
 			(at 150.622 31.75 90)
 			(effects
@@
 			)
 		)
-		(property "Footprint" ""
+		(property "Footprint" "Button_Switch_SMD:SW_SPST_PTS810"
 			(at 137.16 59.69 0)
 			(effects
@@
 			)
 		)
-		(property "Footprint" ""
+		(property "Footprint" "Capacitor_SMD:C_0603_1608Metric"
 			(at 246.0752 55.88 0)
 			(effects
@@
 			)
 		)
-		(property "Footprint" ""
+		(property "Footprint" "Capacitor_SMD:C_0603_1608Metric"
 			(at 153.3652 49.53 0)
 			(effects
@@
 			)
 		)
-		(property "Footprint" ""
+		(property "Footprint" "Resistor_SMD:R_0603_1608Metric"
 			(at 175.26 106.172 90)
 			(effects
@@
 			)
 		)
-		(property "Footprint" ""
+		(property "Footprint" "LED_SMD:LED_0603_1608Metric"
 			(at 182.88 119.38 0)
 			(effects
@@
 			)
 		)
-		(property "Footprint" ""
+		(property "Footprint" "Resistor_SMD:R_0603_1608Metric"
 			(at 155.702 114.3 90)
 			(effects

Commit message: Working on PCB
Parts:
- J1: footprint Connector_USB:USB_Micro-B_Amphenol_10103594-0001LF_Horizontal -> Connector_USB:USB_Micro-B_GCT_USB3076-30-A
Changed lines of the file:
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@@
 			)
 		)
-		(property "Footprint" "Connector_USB:USB_Micro-B_Amphenol_10103594-0001LF_Horizontal"
+		(property "Footprint" "Connector_USB:USB_Micro-B_GCT_USB3076-30-A"
 			(at 72.39 48.26 0)
 			(effects

Commit message: Finished the board
Connections:
- net EN renamed ESP_32EN
Changed lines of the file:
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@@
 		)
 	)
-	(label "EN"
+	(label "ESP_32EN"
 		(at 193.04 60.96 0)
 		(effects
@@
 		)
 	)
-	(label "EN"
+	(label "ESP_32EN"
 		(at 158.75 40.64 0)
 		(effects
