File: tutorial/PhilsLab/60_SwitchingRegulator/EMI_testboard/EMI_testboard.kicad_pcb (KiCad board)
At the start: 2 copper layers, 0 parts

Commit message: BUCK CONVERTER :: Changed capacitors
Parts:
- added C1: 22u, Capacitor_SMD:C_0603_1608Metric, F.Cu at (71.3, 71.3)
- added C2: 100n, Capacitor_SMD:C_0603_1608Metric, F.Cu at (71.3, 73.8)
- added C3: 22u, Capacitor_SMD:C_0603_1608Metric, F.Cu at (87.7, 67.0)
- added C4: 22u, Capacitor_SMD:C_0603_1608Metric, F.Cu at (87.7, 69.5)
- added JP1: SolderJumper_2_Open, Jumper:SolderJumper-2_P1.3mm_Open_TrianglePad1.0x1.5mm, F.Cu at (75.5, 76.4)
- added JP2: SolderJumper_2_Open, Jumper:SolderJumper-2_P1.3mm_Open_TrianglePad1.0x1.5mm, F.Cu at (91.9, 67.5)
- added L1: 47u, Inductor_SMD:L_Neosid_SM-PIC0512H, F.Cu at (85.0, 60.5)
- added R1: 10k, Capacitor_SMD:C_0603_1608Metric, F.Cu at (87.7, 74.5)
- added R2: 24k, Capacitor_SMD:C_0603_1608Metric, F.Cu at (87.7, 77.0)
- added R3: 75k, Capacitor_SMD:C_0603_1608Metric, F.Cu at (87.7, 79.5)
- added U1: ~, Package_TO_SOT_SMD:SOT-23-6, F.Cu at (79.0, 67.0)
