File: tutorial/PhilsLab/60_SwitchingRegulator/EMI_testboard/EMI_testboard.kicad_sch (KiCad schematic)
At the start: 11 parts

Commit message: BUCK CONVERTER :: Changed capacitors
Parts:
- C1, C3, C4: footprint Capacitor_SMD:C_0603_1608Metric -> Capacitor_SMD:C_1210_3225Metric
- L1: footprint Capacitor_SMD:C_0603_1608Metric -> Inductor_SMD:L_Neosid_SM-PIC0512H
Connections:
- net +3V3: now also C3.1, C4.1; no longer C3.2, C4.2
- net GND: now also C3.2, C4.2; no longer C3.1, C4.1
